File: KiCAD/STM32F4xx.sch (KiCad schematic (older format))
At the start: 18 parts

Commit message: Added Power supply filtering and usb port
Parts:
- added C?: 2.2uF, ~, symbol C
- added C? (x11): C, ~, symbol C
- added C? (x2): CP1, ~, symbol CP1
- added C?: 100nF, ~, symbol C
- added C?: 22uF, ~, symbol CP1
- added CR? (x2): CG0603MLC-05LE, symbol ESD
- added F?: MF-MSMF050-2, symbol FUSE-MINI
- added L?: INDUCTOR_SMALL, ~, symbol INDUCTOR_SMALL
- added R? (x2): R, ~, symbol R
- added R? (x2): 22R, ~, symbol R
- added USB?: USBCONN, symbol USBCONN
- C?: value C -> 2.2uF
Connections:
- net labels added: D+, D-, VBUS, VUSB
- wire segments 40 -> 127
Other:
- note added: "Analog power supply"
- note added: "BOOT configuration \n(for enabling the bootloader)"
- note added: "It might be useful to \nmake VSSA to go to\na analog ground plane"
- note added: "NOTE: VBAT is the RTC backup \npower supply, and must lie \nbetween 1.65V and 3.6V\n"
- note added: "Power supply filtering"
- note added: "RESET button"
- note added: "SWD (Serial wire debugging) connector\n"
- note added: "USB Port"
- note added: "USER button"
- moved on the sheet: C?

Commit message: Added serial ports and servo connectors.
Parts:
- added C?: 10uF, ~, symbol C
- added K? (x3): CONN_3, ~, symbol CONN_3
- added P? (x4): CONN_4, ~, symbol CONN_4
- added Q?: FDN340P, ~, symbol MOS_P_DIODE
- added Q? (x3): MOS_N, ~, symbol MOS_N
- added R?: 10K, ~, symbol R
- added R? (x6): R, ~, symbol R
- added U?: XBEE, symbol XBEE
Connections:
- net labels added: +5V, RX1, RX2, RX3, RX4, SERVO1_3V, SERVO1_5V, SERVO2_3V, SERVO2_5V, SERVO3_3V, SERVO3_5V, SERVO_PWR, TX1, TX2, TX3, TX4, Vin, XBEE_ON, XBEE_RESET, XBEE_RX, XBEE_TX
- wire segments 127 -> 262
- no-connect marks 0 -> 15
Other:
- note added: "TODO: The symbol for the mosfet has to be updated to a\nmosfet with diode"
- note added: "USB Power Switch"
- moved on the sheet: C?, CR?, F?, R?, USB?

Commit message: Added buffers for serial ports, dynamixel connector.
Parts:
- removed Q? (x3): MOS_N, ~, symbol MOS_N
- added D? (x4): LED, ~, symbol LED
- added Q? (x3): MOS_N_DIODE, ~, symbol MOS_N_DIODE
- added R? (x4): R, ~, symbol R
- added R?: 10K, ~, symbol R
- added U? (x5): 74AHC2G126, ~, symbol 74AHC2G126
- added U?: DYNAMIXEL_CONN_3, ~, symbol DYNAMIXEL_CONN_3
Connections:
- net labels added: 9.6V_DYN, DATA_DYN, DIR_PORT_DYN, LED1, LED2, LED3, LED4, RX1_3V, RX2_3V, RX3_3V, RX4_3V, RX_DYN, TX1_3V, TX2_3V, TX3_3V, TX4_3V, TX_DYN
- wire segments 262 -> 359
Other:
- note added: "Buffers on the receivers are not needed (5V)"
- note added: "These buffers have to be the 74AHCT2G126 version,\nthe current one won't detect 3v level as high"
- note added: "This has to be inverted"
- note removed: "TODO: The symbol for the mosfet has to be updated to a\nmosfet with diode"
- moved on the sheet: C?, K?, P?, R?, U?

Commit message: Corrected xbee pinout, corrected serial buffers.
Parts:
- removed U? (x4): 74AHC2G126, ~, symbol 74AHC2G126
- added JP? (x4): JUMPER-2, symbol JUMPER-2
- added Q?: MOS_N, ~, symbol MOS_N
- added Q? (x4): MOS_N_DIODE, ~, symbol MOS_N_DIODE
- added R? (x9): R, ~, symbol R
Connections:
- net labels removed: RX1_3V, RX2_3V, RX3_3V, RX4_3V
- wire segments 359 -> 294
Other:
- note added: "DYNAMIXEL servo control"
- note added: "Here I should put some connector for the servo power"
- note added: "LED indicators"
- note added: "SERVO headers"
- note added: "Serial ports to other modules"
- note removed: "Buffers on the receivers are not needed (5V)"
- note removed: "These buffers have to be the 74AHCT2G126 version,\nthe current one won't detect 3v level as high"
- note removed: "This has to be inverted"
- moved on the sheet: C?, CR?, D?, F?, JP?, K?, L?, P?, Q?, R?, SW?, U?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

Commit message: Added IMU.
Parts:
- added C?: 22uF, ~, symbol C
- added C?: 4.7uF, ~, symbol C
- added C?: 10nF, ~, symbol C
- added K?: CONN_3, ~, symbol CONN_3
- added P?: CONN_2, ~, symbol CONN_2
- added Q? (x2): MOS_N_DIODE, ~, symbol MOS_N_DIODE
- added R? (x7): R, ~, symbol R
- added U?: L3GD20, symbol L3GD20
- added U?: LSM303DLHC, symbol LSM303DLHC
Connections:
- net labels added: ACC_INT_1, ACC_INT_2, GYRO_INT_1, GYRO_INT_2, I2C_PCB_SCL, I2C_PCB_SDA, I2C_SCL_PWR_3V, I2C_SCL_PWR_5V, I2C_SDA_PWR_3V, I2C_SDA_PWR_5V, XBEE_SLEEP
- net labels removed: XBEE_ON
- wire segments 294 -> 371
- no-connect marks 15 -> 17
Other:
- note added: "Connector for the power suppy module"
- note added: "IMU"
- note added: "Since this needs 9.6V to work \nI'm currently thinking of breaking\nout the 3 control pins ( Rx, Tx, Dir)\nto connect them to an expansion \nmodule."
- note added: "xBee connector"
- moved on the sheet: C?, CR?, F?, Q?, R?, U?, USB?

Commit message: Added power regulator.
Parts:
- added C?: 1uF X7R 0805, ~, symbol CP1
- added C?: 4.7uF X7R 0805, ~, symbol CP1
- added U?: MCP1825S, ~, symbol MCP1825S
Connections:
- wire segments 371 -> 383
Other:
- note added: "Inertial Measurement Unit (IMU)"
- note added: "LDO Power Regulator\nIn: 5-6V Out: 3V"
- note removed: "IMU"
- moved on the sheet: C?, CR?, D?, F?, JP?, K?, L?, P?, Q?, R?, SW?, U?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

Commit message: Added component values.
Parts:
- removed C?: C, ~, symbol C
- removed R? (x2): R, ~, symbol R
- C? (x11): value C -> 100nF
- C? (x2): value CP1 -> 1uF
- D?: value LED -> BLUE
- D?: value LED -> RED
- D?: value LED -> ORANGE
- D?: value LED -> GREEN
- L?: value INDUCTOR_SMALL -> fcm 0603
- R?: value R -> 100K
- R?: value R -> 220K
- R?: value R -> 47
- R? (x18): value R -> 10K
- R? (x3): value R -> 680
- R?: value R -> 510
- R? (x3): value R -> 4.7K
Connections:
- wire segments 383 -> 488
Other:
- note added: "TODO: Assign interrupts to pins"
- moved on the sheet: C?, D?, JP?, R?, SW?

Commit message: Added ADC connector.
Parts:
- removed R? (x2): R, ~, symbol R
- added K?: CONN_3, ~, symbol CONN_3
- C? (x2): value C -> 20pF
- C?: value C -> 1uF
- R?: value R -> 510
- X?: value CRYSTAL -> 8MHz
Connections:
- net labels added: ADC1, ADC2, ADC3, RX2_3V, RX3_3V, RX4_3V, SPI1_MISO, SPI1_MOSI, SPI1_NSS, SPI1_SCK, T_SWO
- wire segments 488 -> 509
- no-connect marks 17 -> 64
Other:
- note added: "'0' > from flash\n'1' > DFU Mode"
- note added: "ADC connector"
- note removed: "Here I should put some connector for the servo power"
- moved on the sheet: C?, D?, Q?, R?, SW?
