File: KiCAD/STM32F4xx.sch (KiCad schematic (older format))
At the start: 107 parts

Commit message: Finished most of the schematic (except power selection).
Parts:
- removed U?: DYNAMIXEL_CONN_3, ~, symbol DYNAMIXEL_CONN_3
- added P?: CONN_2, ~, symbol CONN_2
Connections:
- net labels added: RX1_3V
- net labels removed: 9.6V_DYN
- wire segments 509 -> 508
Other:
- moved on the sheet: C?, L?, Q?, R?, U?, X?
