File: KiCAD/hebi.sch (KiCad schematic (older format))
At the start: 111 parts, among them K1 CONN_3, K2 CONN_3, K3 CONN_3, K4 CONN_3, K5 CONN_3, P1 CONN_4, P2 CONN_4, P3 CONN_4, P4 CONN_4, P5 CONN_2, P6 CONN_2, Q1 MOS_N_DIODE, Q10 MOS_N_DIODE, Q2 MOS_N_DIODE, Q3 MOS_N_DIODE, Q4 MOS_N_DIODE, Q5 MOS_N_DIODE, Q6 MOS_N_DIODE, Q7 MOS_N_DIODE, Q8 MOS_N, Q9 MOS_N_DIODE, SW1 SW_PUSH, SW2 SW_PUSH, SW3 SW_PUSH, U1 MPU-6050, U2 HMC5883L, U3 MCP1825S, U4 STM32F407VG, U5 XBEE, U6 74AHC2G126, X1 8MHz

Commit message: Removed dynamixel due to spatial requirements (no space left for that)
Parts:
- removed P5: CONN_2, ~, symbol CONN_2
- removed Q8: MOS_N, ~, symbol MOS_N
- removed R29: 10K, ~, symbol R
- removed R30: 4.7K, ~, symbol R
- removed U6: 74AHC2G126, ~, symbol 74AHC2G126
Connections:
- net labels removed: DATA_DYN, DIR_PORT_DYN, RX_DYN, TX_DYN
- wire segments 405 -> 377
- no-connect marks 76 -> 79

Commit message: Routed power tracks, removed IMU.
Parts:
- removed C1, C3: 0.1uF, ~, symbol C
- removed C14: 220nF, ~, symbol C
- removed C2: 10nF, ~, symbol C
- removed C4: 2.2nF, ~, symbol C
- removed C8: 4.7uF, ~, symbol CP1
- removed JP1: JUMPER3, ~, symbol JUMPER3
- removed R4, R9: 4.7K, ~, symbol R
- removed U1: MPU-6050, ~, symbol MPU-6050
- removed U2: HMC5883L, ~, symbol HMC5883L
Connections:
- net labels removed: ACCEL_INT, COMPASS_INT, COMPASS_iNT, I2C_PCB_SCL, I2C_PCB_SDA
- wire segments 377 -> 324
- no-connect marks 79 -> 65
Other:
- note removed: "C1 - Ceramic, X7R, 0.1uF, tol 10%, 4V\nC2 - Ceramic, X7R, 10nF, tol 10%, 4V\nC3 - Ceramic, X7R, 0.1uF, tol 10%, 2V\nC4 - Ceramic, X7R, 2.2, tol 10%, 50V"
- note removed: "Inertial Measurement Unit (IMU)"
